File: batt_main_relay.kicad_sch (KiCad schematic)
At the start: 4 parts, among them J8 Conn_01x90_3Row_Socket, K1 Main Relay, SW00 Key Switch

Commit message: external loops
Parts:
- renumbered SW00 to SW3
Connections:
- net B30: no longer SW3.MP
- net A33 renamed P,E
- net B86 renamed PWR_12V
- no-connect marks 84 -> 85
