File: blank.kicad_sch (KiCad schematic)
At the start: 2 parts, among them J27 Conn_01x90_3Row_Socket

Commit message: external loops
Connections:
- net B23: now also Re11.2 (-); no longer Re11.1 (+)
- net B29: now also J27.86 (B86), Re11.1 (+); no longer J27.29 (B29), Re11.2 (-)
