File: canister_valve.kicad_sch (KiCad schematic)
At the start: 2 parts, among them J26 Conn_01x90_3Row_Socket

Commit message: external loops
Parts:
- renumbered J26 to J28
Connections:
- net B25: now also Re10.2 (-); no longer Re10.1 (+)
- net B29: no longer names the net of J28.29 (B29)
- net B29: no longer Re10.2 (-)
- new net PWR_12V: Re10.1 (+)
- no-connect marks 88 -> 89
