File: fan_control.kicad_sch (KiCad schematic)
At the start: 6 parts, among them J18 Conn_01x90_3Row_Socket, K2 1500A, K3 1502, K4 1500B, M2 Fan1, M3 Fan2

Commit message: external loops
Connections:
- net A33 renamed P,E
- net P,E: no longer J18.33 (A33)
- net B29 renamed PWR_12V
- net PWR_12V: no longer J18.29 (B29)
- no-connect marks 87 -> 89
