File: fuel_pump_relay.kicad_sch (KiCad schematic)
At the start: 2 parts, among them J9 Conn_01x90_3Row_Socket

Commit message: external loops
Connections:
- net B29: no longer names the net of J9.29 (B29)
- net B29: no longer Re1.2 (-)
- net B86 renamed B80
- net B80: now also Re1.2 (-); no longer Re1.1 (+)
- new net PWR_12V: Re1.1 (+)
- no-connect marks 88 -> 89
