File: gas_injector.kicad_sch (KiCad schematic)
At the start: 8 parts, among them J21 Conn_01x90_3Row_Socket

Commit message: external loops
Parts:
- removed J21: Conn_01x90_3Row_Socket, symbol sicma_socket:Conn_01x90_3Row_Socket
- removed LA1: CNG Fuel Type Lamp, symbol Device:Lamp
- removed LA2: High Temp, symbol Device:Lamp
- removed V1: Check Engine-MIL, symbol Device:Lamp
- removed _1, _2, _4: %, symbol Device:Galvanometer
- removed _3: Tr/mn, symbol Device:Galvanometer
- added J27: Conn_01x90_3Row_Socket, symbol sicma_socket:Conn_01x90_3Row_Socket
- added Re6: Gas Inj. 1, symbol Elektuur_1:Re
- added Re7: Gas Inj. 4, symbol Elektuur_1:Re
- added Re8: Gas Inj. 3, symbol Elektuur_1:Re
- added Re9: Gas Inj. 2, symbol Elektuur_1:Re
Connections:
- net PWR_12V: now also Re6.1 (+), Re7.1 (+), Re8.1 (+), Re9.1 (+)
- new net B59: J27.59 (B59), Re8.2 (-)
- new net B60: J27.60 (B60), Re6.2 (-)
- new net B89: J27.89 (B89), Re9.2 (-)
- new net B90: J27.90 (B90), Re7.2 (-)
- no-connect marks 83 -> 86
Other:
- note removed: "0004"
