File: gas_pcd_valve.kicad_sch (KiCad schematic)
At the start: 8 parts, among them J21 Conn_01x90_3Row_Socket

Commit message: external loops
Parts:
- removed J21: Conn_01x90_3Row_Socket, symbol sicma_socket:Conn_01x90_3Row_Socket
- removed LA1: CNG Fuel Type Lamp, symbol Device:Lamp
- removed LA2: High Temp, symbol Device:Lamp
- removed V1: Check Engine-MIL, symbol Device:Lamp
- removed _1, _2, _4: %, symbol Device:Galvanometer
- removed _3: Tr/mn, symbol Device:Galvanometer
- added J27: Conn_01x90_3Row_Socket, symbol sicma_socket:Conn_01x90_3Row_Socket
- added Re11: PCD Valve, symbol Elektuur_1:Re
Connections:
- net PWR_12V: now also Re11.2 (-)
- new net B23: J27.23 (B23), Re11.1 (+)
- no-connect marks 83 -> 89
Other:
- note removed: "0004"
