File: gas_pres_temp.kicad_sch (KiCad schematic)
At the start: 4 parts, among them J13 Conn_01x90_3Row_Socket, U48 GAS Press Rack, U49 Gas Temp Rack, U50 Gas Press Tank

Commit message: external loops
Parts:
- U48: Unit Tag (none) -> 1312A
- U50: Unit Tag (none) -> 1312B
