File: gasoline_injector.kicad_sch (KiCad schematic)
At the start: 8 parts, among them J21 Conn_01x90_3Row_Socket

Commit message: external loops
Parts:
- removed J21: Conn_01x90_3Row_Socket, symbol sicma_socket:Conn_01x90_3Row_Socket
- removed LA1: CNG Fuel Type Lamp, symbol Device:Lamp
- removed LA2: High Temp, symbol Device:Lamp
- removed V1: Check Engine-MIL, symbol Device:Lamp
- removed _1, _2, _4: %, symbol Device:Galvanometer
- removed _3: Tr/mn, symbol Device:Galvanometer
- added J26: Conn_01x90_3Row_Socket, symbol sicma_socket:Conn_01x90_3Row_Socket
- added Re2: Gasoline Inj. 1, symbol Elektuur_1:Re
- added Re3: Gasoline Inj. 4, symbol Elektuur_1:Re
- added Re4: Gasoline Inj. 3, symbol Elektuur_1:Re
- added Re5: Gasoline Inj. 2, symbol Elektuur_1:Re
Connections:
- net PWR_12V: now also Re2.1 (+), Re3.1 (+), Re4.1 (+), Re5.1 (+)
- new net B57: J26.57 (B57), Re4.2 (-)
- new net B58: J26.58 (B58), Re2.2 (-)
- new net B87: J26.87 (B87), Re5.2 (-)
- new net B88: J26.88 (B88), Re3.2 (-)
- no-connect marks 83 -> 86
Other:
- note removed: "0004"
