File: ignation_coils.kicad_sch (KiCad schematic)
At the start: 3 parts, among them J15 Conn_01x90_3Row_Socket

Commit message: external loops
Connections:
- net B86 renamed PWR_12V
- net PWR_12V: no longer J15.86 (B86)
- net P,E renamed GND
- no-connect marks 86 -> 87
