File: injector_valves.kicad_sch (KiCad schematic)
At the start: 9 parts, among them J24 Conn_01x90_3Row_Socket

Commit message: external loops
Connections:
- net B29 renamed PWR_12V
- net PWR_12V: no longer J24.29 (B29)
- no-connect marks 81 -> 82
