File: knock_sensor.kicad_sch (KiCad schematic)
At the start: 2 parts, among them J16 Conn_01x90_3Row_Socket

Commit message: external loops
Parts:
- renumbered C1120 to C113
Connections:
- net A75 renamed GND
