File: oxigen_sensor.kicad_sch (KiCad schematic)
At the start: 3 parts, among them J22 Conn_01x90_3Row_Socket, U53 Oxigen Sensor

Commit message: external loops
Connections:
- net B86 renamed PWR_12V
- net PWR_12V: no longer J22.86 (B86)
- no-connect marks 86 -> 87
