File: speed_sensor.kicad_sch (KiCad schematic)
At the start: 2 parts, among them J25 Conn_01x90_3Row_Socket, U54 Vehicle Speed Sensor

Commit message: external loops
Parts:
- renumbered J25 to J31
Connections:
- net B86: no longer names the net of J31.86 (B86)
- net B86: no longer U54.1 (V_{CC})
- new net PWR_12V: U54.1 (V_{CC})
- no-connect marks 88 -> 89
