File: fan_control_AC.kicad_sch (KiCad schematic)
At the start: 3 parts, among them J20 Conn_01x90_3Row_Socket, U51 MCP9700Ax-ETT, U52 TMAP

Commit message: external loops
Parts:
- removed J20: Conn_01x90_3Row_Socket, symbol sicma_socket:Conn_01x90_3Row_Socket
- removed U51: MCP9700Ax-ETT, Package_TO_SOT_SMD:SOT-23, symbol Sensor_Temperature:MCP9700Ax-ETT
- removed U52: TMAP, symbol Sensor_Pressure:MPXHZ6115A
- added J18: Conn_01x90_3Row_Socket, symbol sicma_socket:Conn_01x90_3Row_Socket
- added K2: 1500A, PCM_SparkFun-Electromechanical:Relay_SPDT_20A_27.6x32.0mm, symbol SparkFun-Electromechanical:Relay_SPDT_20A_5V_27.6x32.0mm
- added K3: 1502, PCM_SparkFun-Electromechanical:Relay_SPDT_20A_27.6x32.0mm, symbol SparkFun-Electromechanical:Relay_SPDT_20A_5V_27.6x32.0mm
- added K4: 1500B, PCM_SparkFun-Electromechanical:Relay_SPDT_20A_27.6x32.0mm, symbol SparkFun-Electromechanical:Relay_SPDT_20A_5V_27.6x32.0mm
- added M2: Fan1, symbol Motor:Fan
- added M3: Fan2, symbol Motor:Fan
- added Re130: AC Compressor Relay, symbol Elektuur_1:Re
- added Re131: AC Compressor Control Relay, symbol Elektuur_1:Re
Connections:
- new net: K3.4, K4.5, M3.1 (+)
- new net: K3.3, M2.2 (-)
- new net A42: J18.42 (A42), Re131.1 (+)
- new net A71: J18.71 (A71), K2.5, M2.1 (+)
- new net B20: J18.20 (B20), K3.1, K4.1
- new net B50: J18.50 (B50), K2.1
- new net B79: J18.79 (B79), Re130.2 (-)
- new net P,E: K3.5, M3.2 (-)
- new net PWR_12V: K2.2, K2.3, K3.2, K4.2, K4.3, Re130.1 (+), Re131.2 (-)
- no-connect marks 86 -> 87

Commit message: external loops arrangments1
Parts:
- added SW5: SW_MEC_5G, symbol Switch:SW_MEC_5G
Connections:
- net P,E: now also SW5.3 (B), SW5.4 (B)
- net at J18.5 (A5): now also SW5.1 (A), SW5.2 (A)
- no-connect marks 87 -> 86
