File: cng_switch.kicad_sch (KiCad schematic)
At the start: 8 parts, among them J21 Conn_01x90_3Row_Socket

Commit message: external loops
Parts:
- removed J21: Conn_01x90_3Row_Socket, symbol sicma_socket:Conn_01x90_3Row_Socket
- removed LA1: CNG Fuel Type Lamp, symbol Device:Lamp
- removed LA2: High Temp, symbol Device:Lamp
- removed V1: Check Engine-MIL, symbol Device:Lamp
- removed _1, _2, _4: %, symbol Device:Galvanometer
- removed _3: Tr/mn, symbol Device:Galvanometer
- added J30: Conn_01x90_3Row_Socket, symbol sicma_socket:Conn_01x90_3Row_Socket
- added SW4: CNG Switch, symbol Switch:SW_MEC_5G
Connections:
- new net A64: J30.64 (A64), SW4.1 (A), SW4.2 (A)
- new net P,E: SW4.3 (B), SW4.4 (B)
- no-connect marks 83 -> 89
Other:
- note removed: "0004"

Commit message: air conditioner updated
Connections:
- net P,E renamed PWR_12V
