File: communications.kicad_sch (KiCad schematic)
At the start: 3 parts, among them J23 Conn_01x90_3Row_Socket

Commit message: external loops
Parts:
- removed R137, R138: 120, Resistor_SMD:R_0603_1608Metric, symbol Device:R_Small
- added J24: OBD, symbol Connector:DA15_Pins
- added J25: Immobilizer, symbol Connector:Conn_01x01_Pin
Connections:
- net B53: now also J25.1 (Pin_1)
- net B76: now also J24.14 (P14)
- net B77: now also J24.6
- net B78: now reaches J23.78 (B78)
- net B78: now also J24.7
- net A64: no longer names the net of J23.64 (A64)
- no-connect marks 86 -> 98
Other:
- note added: "Twisted Pair"

Commit message: communications updated
Parts:
- removed J24: OBD, symbol Connector:DA15_Pins
- removed J25: Immobilizer, symbol Connector:Conn_01x01_Pin
- added J24: Immobilizer, symbol Connector_Generic:Conn_01x02
- added M4: OBDII, OBDII, symbol Connectors:OBDII
Connections:
- net B53: now also J24.2 (Pin_2)
- net B76: now also M4.14 (CANLOW)
- net B77: now also M4.6 (CANHIGH)
- net B78: now also M4.7 (ISOK-LINE)
- new net: J24.1 (Pin_1), M4.15 (ISOL-LINE)
- new net GND: M4.4 (CHASGND)
- new net PWR_12V: M4.16 (BATTPOWER)
- no-connect marks 98 -> 96
